File: kicad/SCNano-Main-PcbDoc.kicad_pcb (KiCad board)
At the start: 2 copper layers, 164.7 x 98 mm, 26 parts, among them CON1 Grove 4 Pin Connector Female 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, IC1 Dual 4-Channel Analog Multipl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, J1 DC Jack, 1.0 x 3.4 mm (for 1.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, Q1 MOSFET N-channel 30V (the eas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, Q2 MOSFET N-channel 30V (the eas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, Q3 MOSFET N-channel 30V (the eas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, Q4 MOSFET N-channel 30V (the eas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, SW1 SWITCH SLIDE DPDT 200MA 30V

Commit message: Altium Class Name directives are unsupported in KiCAD. The conversion process placed the same ClassName directives as labels, which caused multiple nets to be treated as the same net.  Changed those labels into texts.
Parts:
- ANT1: value Antenna, Cellular Radio, 3G -> 3G Antenna
- BAT1: value Battery Holder, 2x18650, T/H -> KEYSTONE_1049
- BOM1: value Additional BOM Item -> Battery - 1of 2
- BOM2: value Additional BOM Item -> Battery - 2 of 2
- C1: value Polarized Capacitor (Radial) -> CAP POL RB13-25
- CON1: value Grove 4 Pin Connector Female T/H, labeled for Safecast Geiegie products -> SC_CON_GEIGIE_4PIN
- IC1: value Dual 4-Channel Analog Multiplexer/Demultiplexer DIP-16 -> SN74LV4052A
- J1: value DC Jack, 1.0 x 3.4 mm (for 1.1 x 3.5 mm plug). T/H -> ~
- MOD1: value Adafruit DC / Solar Lithium Ion/Polymer charger - v2 -> LiPo Charger
- MOD2: value Adafruit FONA 3G Cellular + GPS Breakout -> FONA 3G
- MOD3: value Adafruit INA219 High Side DC Current Sensor Breakout -> Current Sensor
- MOD4: value Adafruit high-resolution ultra low-power triaxial (3-axis) accelerometer module (LIS3DH) -> 3-Axis
- MOD5: value Adafruit Ultimate GPS Breakout - 66 channel w/10 Hz updates - Version 3 -> GPS
- MOD6: value Redbear Nano V2 Plus - nRF52832 processor module -> Nano V2
- MOD7: value Redbear DAPLink 1.5 (included in purchase with BLE Nano) -> DAPLink 1.5
- MOD8: value Adafruit 1833 MicroUSB Breakout Module -> MicroUSB
- OLED1: value IIC 0.96" Inches White I2C 128x64 OLED LCD Display Module, with VCC on pin 1 -> OLED 128x64
- Q1, Q2, Q3, Q4: value MOSFET N-channel 30V (the easy to handle IPAK version) carefully chosen for high-current Fona, and is a very flexible p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 -> STU85N3LH5
- SOLARPANEL1: value 1 Watt Solar Panel -> VOLTAIC_SOLAR_PANEL_1W
- SW1: value SWITCH SLIDE DPDT 200MA 30V -> SW-DPDT
- VREG1: value Pololu 3.3V Step-Up/Step-Down Voltage Regulator Module (S7V8F3) -> Regulator 3.3V
- VREG2: value Pololu Adjustable Boost Regulator Module (2.5-9.5V) -> Regulator Variable
Connections:
- net BAT-BUS renamed /BAT-BUS
- net BAT-POS renamed /BAT-POS
- net BAT-SW renamed /BAT-SW
- net ENABLE-CELL renamed /ENABLE-CELL
- net ENABLE-GEIG renamed /ENABLE-GEIG
- net ENABLE-GPS renamed /ENABLE-GPS
- net ENABLE_TWI renamed /ENABLE_TWI
- net FONA-BAT renamed /FONA-BAT
- net FONA-RX renamed /FONA-RX
- net FONA-TX renamed /FONA-TX
- net GEIGER0 renamed /GEIGER0
- net GEIGER1 renamed /GEIGER1
- net GND-CELL renamed /GND-CELL
- net GND-GEIG renamed /GND-GEIG
- net GND-GPS renamed /GND-GPS
- net GND-TWI renamed /GND-TWI
- net LIS-INT renamed /LIS-INT
- net MCU-RX renamed /MCU-RX
- net MCU-SWCLK renamed /MCU-SWCLK
- net MCU-SWDIO renamed /MCU-SWDIO
- net MCU-TX renamed /MCU-TX
- net NANO_VIN renamed /NANO_VIN
- net NetC1_1 renamed Net-(C1-Pad1)
- net PANEL-POS renamed /PANEL-POS
- net TWI-SCL renamed /TWI-SCL
- net TWI-SDA renamed /TWI-SDA
- net UGPS-RX renamed /UGPS-RX
- net UGPS-TX renamed /UGPS-TX
- IC1 pad 1: (no net) -> Net-(IC1-Pad1)
- IC1 pad 11: (no net) -> Net-(IC1-Pad11)
- IC1 pad 12: (no net) -> Net-(IC1-Pad12)
- IC1 pad 4: (no net) -> Net-(IC1-Pad4)
- J1 pad 3: (no net) -> Net-(J1-Pad3)
- MOD1 pad 7: (no net) -> Net-(MOD1-Pad7)
- MOD2 pad 1: (no net) -> Net-(MOD2-Pad1)
- MOD2 pad 10: (no net) -> Net-(MOD2-Pad10)
- MOD2 pad 12: (no net) -> Net-(MOD2-Pad12)
- MOD2 pad 13: (no net) -> Net-(MOD2-Pad13)
- MOD2 pad 14: (no net) -> Net-(MOD2-Pad14)
- MOD2 pad 15: (no net) -> Net-(MOD2-Pad15)
- MOD2 pad 16: (no net) -> Net-(MOD2-Pad16)
- MOD2 pad 17: (no net) -> Net-(MOD2-Pad17)
- MOD2 pad 18: (no net) -> Net-(MOD2-Pad18)
- MOD2 pad 8: (no net) -> Net-(MOD2-Pad8)
- MOD2 pad 9: (no net) -> Net-(MOD2-Pad9)
- MOD4 pad 1: (no net) -> Net-(MOD4-Pad1)
- MOD4 pad 6: (no net) -> Net-(MOD4-Pad6)
- MOD4 pad 7: (no net) -> Net-(MOD4-Pad7)
- MOD5 pad 1: (no net) -> Net-(MOD5-Pad1)
- MOD5 pad 2: (no net) -> Net-(MOD5-Pad2)
- MOD5 pad 3: (no net) -> Net-(MOD5-Pad3)
- MOD5 pad 4: (no net) -> Net-(MOD5-Pad4)
- MOD5 pad 9: (no net) -> Net-(MOD5-Pad9)
- MOD8 pad 2: (no net) -> Net-(MOD8-Pad2)
- MOD8 pad 3: (no net) -> Net-(MOD8-Pad3)
- MOD8 pad 4: (no net) -> Net-(MOD8-Pad4)
- SW1 pad 3: (no net) -> Net-(SW1-Pad3)
- VREG1 pad 4: (no net) -> Net-(VREG1-Pad4)
Routing:
- added copper zone on F.Cu, net NetC1_1
- added copper zone on B.Cu, net PANEL-POS
- added copper zone on F.Cu, net PANEL-POS
- removed copper zone on B.Cu, net /PANEL-POS
- removed copper zone on F.Cu, net /PANEL-POS
- removed copper zone on F.Cu, net Net-(C1-Pad1)
